Commit message: Setup of door env

File: objects/board_easy.urdf (robot description, URDF)
Before this commit: robot board, 2 links, 1 joints
Links:
- removed link circle
- added link target, mass 0
Joints:
- joint board__circle: child circle -> target

File: objects/door.urdf (robot description, URDF)
Before this commit: robot door, 3 links, 2 joints
Links:
- link base_link: mass 2.168 -> 5; geometry collision box size=0.1 0.05 0.5; collision box size=0.1 0.05 0.5
- link door_link: mass 3.354 -> 2; geometry collision box size=0.01 0.4 0.51
- link handle_link: mass 0.56914 -> 0.2; geometry collision box size=0.02 0.15 0.01; collision cylinder length=0.06 radius=0.01
Joints:
- removed joint base__door
- removed joint door__handle
- added joint handle_joint: type revolute, parent door_link, child handle_link, origin xyz=-0.01 0.35 0 rpy=3.145 0 0, axis 1 0 0, limit lower=0 upper=0.7854 effort=100 velocity=1
- added joint hinge_joint: type revolute, parent base_link, child door_link, origin xyz=-0.05 -0.2 0.25 rpy=0 0 0, axis 0 0 1, limit lower=0 upper=1.5708 effort=1 velocity=1
