Commit message: Added sliding door environment

File: objects/sliding_door.urdf (robot description, URDF)
Before this commit: robot door, 3 links, 2 joints
Links:
- link base_link: geometry collision box size=0.02 0.4 0.45; collision box size=0.1 0.05 0.45
- link door_link: geometry collision box size=0.02 0.4 0.45
- link handle_link: geometry collision box size=0.02 0.02 0.16; collision box size=0.06 0.02 0.02
Joints:
- removed joint hinge_joint
- added joint door_joint: type prismatic, parent base_link, child door_link, origin xyz=-0.03 0.2 0.25 rpy=0 0 0, axis 0 -1 0, limit lower=0 upper=0.4 effort=1 velocity=1
- joint handle_joint: axis 1 0 0 -> (none); limit lower=0 upper=0.7854 effort=100 velocity=1 -> (none); origin xyz=-0.01 0.35 0 rpy=3.145 0 0 -> xyz=-0.01 -0.16 0 rpy=0 0 0; type revolute -> fixed
