Commit message: created new sliding door scenario with lose parts

File: objects/hatch_door.urdf (robot description, URDF)
Before this commit: robot sliding_door, 3 links, 2 joints
Links:
- removed link base_link
- link door_link: mass 0.5 -> 5; geometry collision box size=0.018 0.29 0.02; collision box size=0.018 0.29 0.02
Joints:
- removed joint door_joint
- joint handle_joint: origin xyz=-0.01 -0.12 0 rpy=0 0 0 -> xyz=0 -0.12 0.01 rpy=0 1.57 0

Commit message: Made sliding door heavier for greater force readings

File: objects/hatch_door.urdf (robot description, URDF)
Before this commit: robot hatch_door, 2 links, 1 joints
Links:
- link door_link: mass 5 -> 50

Commit message: Added more variations on BOPT training

File: objects/hatch_door.urdf (robot description, URDF)
Before this commit: robot hatch_door, 2 links, 1 joints
Links:
- link handle_link: geometry collision box size=0.05 0.02 0.02; collision box size=0.05 0.02 0.02
